File: supersmymps v2.kicad_sch (KiCad schematic)
At the start: 86 parts, among them J1 c21 socket, J2 Wire, J3 Conn_01x03_Socket, Q1 IRFP360, Q2 IRFP360, Q3 IRFP360, Q4 IRFP360, Q5 IRFP360, T1 Transformer_1P_2S, U1 BS1212S, U2 TL494, U3 TLV5638, U4 TLP421P, U5 TLP421P, U6 FAN7382, U7 FAN7382

Commit message: Add files via upload
Lets take a moment to brake the ice, so my intentions are known
Parts:
- removed A1: Arduino_Nano_v3.x, Module:Arduino_Nano, symbol MCU_Module:Arduino_Nano_v3.x
- removed C17, C18: 10000u, Capacitor_THT:CP_Radial_D30.0mm_P10.00mm_SnapIn, symbol Device:C_Polarized
- removed D7, D8: S30D45C, Package_TO_SOT_THT:TO-247-3_Vertical, symbol Device:D_Schottky_Dual_CommonCathode_AKA_Parallel
- added BZ1: Buzzer, Buzzer_Beeper:Buzzer_12x9.5RM7.6, symbol Device:Buzzer
- added C19, C20, C22, C23, C25, C26, C27, C28: 100u/63V, Capacitor_THT:CP_Radial_D8.0mm_P3.50mm, symbol Device:C_Polarized
- added C2, C3: 10n, Capacitor_THT:C_Disc_D5.0mm_W2.5mm_P2.50mm, symbol Device:C
- added C21: 220u/6.3V, Capacitor_THT:CP_Radial_D6.3mm_P2.50mm, symbol Device:C_Polarized
- added C24: 1u/10V, Capacitor_THT:C_Disc_D5.0mm_W2.5mm_P5.00mm, symbol Device:C
- added C29: 470u/16V, Capacitor_THT:CP_Radial_D8.0mm_P3.50mm, symbol Device:C_Polarized
- added D11: IN4002, Diode_THT:D_A-405_P7.62mm_Horizontal, symbol Device:D
- added D12: 12V, Diode_THT:D_A-405_P7.62mm_Horizontal, symbol Device:D_Zener
- added D2: BAT48RL, Diode_THT:D_DO-35_SOD27_P7.62mm_Horizontal, symbol Diode:BAT48RL
- added J2: programmer, Connector_PinHeader_2.54mm:PinHeader_1x06_P2.54mm_Vertical, symbol Connector:Conn_01x06_Socket
- added J3: Front_Panel, Connector_IDC:IDC-Header_2x10_P2.54mm_Vertical, symbol Connector_Generic:Conn_02x10_Counter_Clockwise
- added L3, L5: 3.2u, Inductor_THT:L_Toroid_Vertical_L22.4mm_W10.2mm_P7.90mm_Vishay_TJ4, symbol Device:L
- added L4: 3.958u, Inductor_THT:L_Toroid_Vertical_L22.4mm_W10.2mm_P7.90mm_Vishay_TJ4, symbol Device:L
- added Q6: IRFZ44N, Package_TO_SOT_THT:TO-220-3_Vertical, symbol Transistor_FET:IRF3205
- added Q7: IRFP3006, Package_TO_SOT_THT:TO-247-3_Vertical, symbol Transistor_FET:IRFP4468PbF
- added Q8: MPSA42, Package_TO_SOT_THT:TO-92_Inline_Wide, symbol Transistor_BJT:MPSA42
- added R1: 330k, Resistor_THT:R_Axial_DIN0207_L6.3mm_D2.5mm_P10.16mm_Horizontal, symbol Device:R
- added R12: 910k, Resistor_THT:R_Axial_DIN0207_L6.3mm_D2.5mm_P10.16mm_Horizontal, symbol Device:R
- added R13: 15k, Resistor_THT:R_Axial_DIN0207_L6.3mm_D2.5mm_P10.16mm_Horizontal, symbol Device:R
- added R14: 220, Resistor_THT:R_Axial_DIN0207_L6.3mm_D2.5mm_P10.16mm_Horizontal, symbol Device:R
- added R15, R16, R17, R18: 300m, Resistor_SMD:R_2512_6332Metric_Pad1.40x3.35mm_HandSolder, symbol Device:R
- added R2: 4.7k, Resistor_THT:R_Axial_DIN0207_L6.3mm_D2.5mm_P10.16mm_Horizontal, symbol Device:R
- added R28, R31: 330, Resistor_THT:R_Axial_DIN0207_L6.3mm_D2.5mm_P10.16mm_Horizontal, symbol Device:R
- added R29, R30: 10k, Resistor_THT:R_Axial_DIN0204_L3.6mm_D1.6mm_P5.08mm_Horizontal, symbol Device:R
- added R32: 1/5W, Resistor_THT:R_Axial_Power_L38.0mm_W6.4mm_P40.64mm, symbol Device:R
- added R33: 1k, Resistor_THT:R_Axial_DIN0204_L3.6mm_D1.6mm_P5.08mm_Horizontal, symbol Device:R
- added R5: 3.3, Resistor_THT:R_Axial_DIN0207_L6.3mm_D2.5mm_P10.16mm_Horizontal, symbol Device:R
- added RV1: 10k, Potentiometer_THT:Potentiometer_Bourns_3296W_Vertical, symbol Device:R_Potentiometer
- added U10: LM1117DT-5.0, Package_TO_SOT_SMD:TO-252-3_TabPin2, symbol Regulator_Linear:LM1117DT-5.0
- added U11: IL300, symbol Isolator_Analog:IL300
- added U12, U13: TLP421P, Package_DIP:DIP-4_W7.62mm, symbol Isolator:TLP785
- added U2: ICE1PCS02, Package_DIP:DIP-8_W7.62mm, symbol Regulator_Controller:ICE1PCS02
- added U7: PIC16F18455-I/SO, Package_SO:SOIC-28W_7.5x17.9mm_P1.27mm, symbol MCU_Microchip_PIC16:PIC16F1786-xSO
- C1: value 1u -> 1u/50V
- C18: renamed from C7; value 1u -> 470u/16V; footprint Capacitor_THT:CP_Radial_D4.0mm_P1.50mm -> Capacitor_THT:CP_Radial_D8.0mm_P3.50mm
- C8: renamed from C6; value 6.8u -> 6.8u/400V
- C9: renamed from C8; value 470u -> 470u/400V
- D10: renamed from D9; value S40D45C -> S60SC6MT
- D6: renamed from D5; value S30D45C -> S60SC6MT
- D7: renamed from D6; value S30D45C -> S60SC6MT
- H4: renamed from H6; value + connection to load -> +
- H5: renamed from H7; value - connection to shunt -> -; now in the parts list
- J5: renamed from J2; value Wire -> Wire (it's copper)
- L2: value 5u -> 3.2u; footprint Inductor_THT:L_Toroid_Vertical_L41.9mm_W19.1mm_P15.80mm_Vishay_TJ7 -> Inductor_THT:L_Toroid_Vertical_L22.4mm_W10.2mm_P7.90mm_Vishay_TJ4
- R19: renamed from R9; value 100 -> 330
- R20: renamed from R10; value 100 -> 330
- load1: now left out of the parts list
- renumbered C9 to C10, C10 to C11, C11 to C12, C12 to C13, C13 to C14, C14 to C15, C15 to C16, C16 to C17, C2 to C4, C3 to C5, C4 to C6, C5 to C7, D2 to D3, D3 to D4, D4 to D5, H3 to H1, H1 to H2, H2 to H3, J3 to J4, R6 to R10, R7 to R11, R11 to R21, R12 to R22, R13 to R23, R14 to R24, R15 to R25, R16 to R26, R17 to R27, R1 to R3, R2 to R4, R4 to R6, R5 to R7, R3 to R9, RV1 to RV2, RV2 to RV3, TP5 to TP4, TP4 to TP5, U2 to U4, U4 to U5, U5 to U6, U6 to U8, U7 to U9
Connections:
- net GNDD is gone; now on net GND: C10.2, C11.2, R21.2, R22.2, U1.3 (GNDOUT), U8.4 (COM), U9.4 (COM)
- net +12V: now also D11.2 (A), J3.15 (Pin_15), R29.1, U10.3 (VI), U13.4
- net +12VA: now also U2.7 (VCC)
- net +5V: now also C21.1, D2.1 (K), J3.20 (Pin_20), U10.2 (VO), U7.20 (V_{DD})
- net 2IN+: now also JP2.2 (B), JP6.2 (B)
- net 300V clean: now also R1.1, R12.1
- net GND: now also C2.2, C3.2, R13.1, R15.2, R16.2, R17.2, R18.2, R2.2, U2.1 (GND); no longer D1.3 (-)
- net GND1: now also BZ1.2 (+), C19.2, C20.2, C21.2, C22.2, C23.2, C25.2, C26.2, C27.2, C28.2, J2.3 (Pin_3), J3.10 (Pin_10), J3.17 (Pin_17), Q6.3 (S), Q8.1 (E), R28.2, R30.2, R31.2, U10.1 (GND), U12.3, U7.19 (V_{SS}), U7.8 (V_{SS})
- net PFC1: now also R5.2
- net VBUS: now also C23.1, C24.2, C25.1, L4.2, Q7.2 (D), R32.2; no longer H4.1, JP4.1 (A), JP7.1 (A), L2.2, load1.1
- net DAC_~{CS}: now reaches TP5.1, U3.3 (~{CS})
- net DAC_~{CS}: now also U7.15 (RC4)
- net live filtered: now reaches D1.2, FL1.2
- net neut filtered: now reaches D1.4, FL1.4
- net -HALF_RECT: now reaches D7.2 (A)
- net -HALF_RECT: now also D10.3 (K)
- net rectified 300V: now reaches C8.1, D1.1 (+), L1.1
- net SPI_MOSI: now reaches TP3.1, U3.1 (DIN)
- net SPI_MOSI: now also J3.16 (Pin_16), U7.16 (RC5)
- net SPI_CLK: now reaches TP4.1, U3.2 (SCLK)
- net SPI_CLK: now also J3.18 (Pin_18), U7.14 (RC3)
- net +HALF_RECT: now reaches D6.2 (A)
- net +HALF_RECT: now also D10.1 (K)
- net at L2.1: now also C22.1, C28.1, L5.2; no longer D10.2 (A)
- net LINE renamed VAC
- net set to 750 ohm: no longer names the net of RV3.1
- new net: D2.2 (A), J2.2 (Pin_2)
- new net: Q6.1 (G), R30.1, U13.3
- new net: Q8.2 (B), R29.2, U12.4
- new net: C19.1, C27.1, L2.2, L3.1
- new net: R28.1, U12.2
- new net: C29.1, D11.1 (K), R33.1
- new net: C20.1, C24.1, C26.1, L3.2, L4.1
- new net: R2.1, RV1.3
- new net: D12.1 (K), Q7.1 (G), Q8.3 (C), R33.2
- new net: R5.1, U2.8 (GATE)
- new net: R31.1, U13.2
- new net: C2.1, U2.2 (ICOMP)
- new net: RV1.2, U2.4 (VINS)
- new net: C3.1, U2.5 (VCOMP)
- new net: R12.2, R13.2, U2.6 (VSENSE)
- new net: R1.2, RV1.1
- new net: Q6.2 (D), R32.1
- new net 7SEG_A: J3.5 (Pin_5), U7.21 (RB0)
- new net 7SEG_B: J3.6 (Pin_6), U7.22 (RB1)
- new net 7SEG_C: J3.7 (Pin_7), U7.23 (RB2)
- new net 7SEG_D: J3.8 (Pin_8), U7.24 (RB3)
- new net 7SEG_DEMUX_A: J3.1 (Pin_1), U7.6 (RA4)
- new net 7SEG_DEMUX_B: J3.2 (Pin_2), U7.7 (RA5)
- new net 7SEG_DEMUX_C: J3.3 (Pin_3), U7.10 (RA6)
- new net 7SEG_DEMUX_D: J3.4 (Pin_4), U7.9 (RA7)
- new net ADC0: U7.2 (RA0)
- new net ADC1: U7.3 (RA1)
- new net BUZZER: BZ1.1 (-), U7.5 (RA3)
- new net CROWBAR: U13.1, U7.4 (RA2)
- new net DISPLAY_~{CS}: J3.19 (Pin_19), U7.17 (RC6)
- new net FAN_PWM: J3.14 (Pin_14), U7.12 (RC1)
- new net ICSPCLK: J2.5 (Pin_5), U7.27 (ICSPCLK/RB6)
- new net ICSPDAT: J2.4 (Pin_4), U7.28 (ICSPDAT/RB7)
- new net LV_RECT: D10.2 (A), L5.1
- new net OUTPUT_CONTROL: U12.1, U7.11 (RC0)
- new net PFC_ISENSE: R14.2, U2.3 (ISENSE)
- new net PFC_SHUNT: D1.3 (-), R14.1, R15.1, R16.1, R17.1, R18.1
- new net UI_0: J3.9 (Pin_9), U7.25 (RB4)
- new net UI_1: J3.11 (Pin_11), U7.26 (RB5)
- new net UI_2: J3.12 (Pin_12), U7.18 (RC7)
- new net UI_3: J3.13 (Pin_13), U7.13 (RC2)
- new net VDC: C29.2, D12.2 (A), H4.1, JP4.1 (A), JP7.1 (A), Q7.3 (S), load1.1
- new net VPP: J2.1 (Pin_1), U7.1 (RE3/~{MCLR}/V_{PP})
- no-connect marks 2 -> 3
Other:
- note added: "AC INPUT"
- note added: "CROWBAR"
- note added: "DAC"
- note added: "DC OUTPUT"
- note added: "EXTERNAL CONNECTORS"
- note added: "FULL BRIDGE RECTIFIER"
- note added: "GALVANIC ISOLATION SUPPLY"
- note added: "LV OUTPUT FILTER"
- note added: "MICROCONTROLLER UNIT"
- note added: "POWER FACTOR CORRECTION"
- note added: "POWER FACTOR CORRECTION CONTROL"
- note added: "POWER SWITCHING"
- note added: "POWER SWITCHING CONTROL"
- note added: "SPI CLK"
- note added: "SPI DAC ~{CS}"
- note added: "SPI DISPLAY ~{CS}"
- note added: "SPI OUT"
- note added: "master clear with internal pullup"
- note added: "set to 750 ohm"
- note added: "use internal 24Mhz/30Mhz crystal setting"
- moved on the sheet: C1, C10, C11, C12, C13, C14, C15, C16, C17, C18, C7, C8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
