File: supersmymps v2.kicad_sch (KiCad schematic)
At the start: 129 parts, among them J1 c21 socket, J2 programmer, J3 Front_Panel, J4 Conn_01x03_Socket, J5 Wire (it's copper), Q1 IRFP360, Q2 IRFP360, Q3 IRFP360, Q4 IRFP360, Q5 IRFP360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

Commit message: Add files via upload
Parts:
- added C31: 1u/50V, Capacitor_THT:CP_Radial_D4.0mm_P1.50mm, symbol Device:C_Polarized
- added C32, C33: 1u, Capacitor_THT:CP_Radial_D4.0mm_P1.50mm, symbol Device:C_Polarized
Connections:
- net +12V: now also C32.1
- net GND1: now also C31.2, C32.2, C33.2
- net VPP: now also C31.1
- net REF: now reaches TP1.1, U3.6 (REF)
- net REF: now also U4.13 (OUTCTRL), U4.14 (REF), C33.1
Other:
- note added: "DIGITAL-TO-ANALOG CONVERTER"
- note removed: "DAC"
- moved on the sheet: TP1, TP2, TP3, TP4, TP5, U1, U3
