File: supersmymps v2.kicad_pcb (KiCad board)
At the start: 2 copper layers, 200 x 140 mm, 88 parts, among them J2 Wire, J3 Conn_01x03_Socket, Q1 IRFP360, Q2 IRFP360, Q3 IRFP360, Q4 IRFP360, Q5 IRFP360, T1 Transformer_1P_2S, U1 BS1212S, U2 TL494, U3 TLV5638, U4 TLP421P, U5 TLP421P, U6 FAN7382, U7 FAN7382

Commit message: Add files via upload
Lets take a moment to brake the ice, so my intentions are known
Parts:
- removed A1: Arduino_Nano_v3.x, Module:Arduino_Nano
- removed the C17 at (198.0, 58.1)
- removed the C18 at (208.0, 88.6)
- removed the D7 at (143.2, 36.5)
- removed D8: S30D45C, Package_TO_SOT_THT:TO-247-3_Vertical
- removed H7: output -, MountingHole:MountingHole_5.3mm_M5_Pad
- removed TP1: REF_DAC, TestPoint:TestPoint_Pad_D2.0mm
- removed TP2: GND1, TestPoint:TestPoint_Pad_D2.0mm
- removed TP3: DIN_DAC, TestPoint:TestPoint_Pad_D2.0mm
- removed TP4: CS_DAC, TestPoint:TestPoint_Pad_D2.0mm
- removed TP5: CLK_DAC, TestPoint:TestPoint_Pad_D2.0mm
- added BZ1: Buzzer, Buzzer_Beeper:Buzzer_12x9.5RM7.6, F.Cu at (185.9, 123.4)
- added C19: 100u/63V, Capacitor_THT:CP_Radial_D8.0mm_P3.50mm, F.Cu at (178.3, 70.0)
- added C2: 10n, Capacitor_THT:C_Disc_D5.0mm_W2.5mm_P2.50mm, F.Cu at (28.9, 147.8)
- added C20: 100u/63V, Capacitor_THT:CP_Radial_D8.0mm_P3.50mm, F.Cu at (178.3, 60.5)
- added C21: 220u/6.3V, Capacitor_THT:CP_Radial_D6.3mm_P2.50mm, F.Cu at (129.2, 102.7)
- added C22: 100u/63V, Capacitor_THT:CP_Radial_D8.0mm_P3.50mm, F.Cu at (188.3, 83.4)
- added C23: 100u/63V, Capacitor_THT:CP_Radial_D8.0mm_P3.50mm, F.Cu at (171.7, 38.4)
- added C24: 1u/10V, Capacitor_THT:C_Disc_D5.0mm_W2.5mm_P5.00mm, F.Cu at (202.1, 44.5)
- added C25: 100u/63V, Capacitor_THT:CP_Radial_D8.0mm_P3.50mm, F.Cu at (162.4, 38.4)
- added C26: 100u/63V, Capacitor_THT:CP_Radial_D8.0mm_P3.50mm, F.Cu at (178.3, 51.2)
- added C27: 100u/63V, Capacitor_THT:CP_Radial_D8.0mm_P3.50mm, F.Cu at (178.3, 79.4)
- added C28: 100u/63V, Capacitor_THT:CP_Radial_D8.0mm_P3.50mm, F.Cu at (188.3, 92.8)
- added C29: 470u/16V, Capacitor_THT:CP_Radial_D8.0mm_P3.50mm, F.Cu at (212.1, 49.8)
- added C3: 10n, Capacitor_THT:C_Disc_D5.0mm_W2.5mm_P2.50mm, F.Cu at (51.5, 156.0)
- added D11: IN4002, Diode_THT:D_A-405_P7.62mm_Horizontal, F.Cu at (210.7, 34.3)
- added D12: 12V, Diode_THT:D_A-405_P7.62mm_Horizontal, F.Cu at (211.8, 43.6)
- added D2: BAT48RL, Diode_THT:D_DO-35_SOD27_P7.62mm_Horizontal, F.Cu at (137.9, 106.7)
- added H5: -, MountingHole:MountingHole_5.3mm_M5_Pad, F.Cu at (161.5, 27.4)
- added J2: programmer, Connector_PinHeader_2.54mm:PinHeader_1x06_P2.54mm_Vertical, F.Cu at (140.4, 117.3)
- added J3: Front_Panel, Connector_IDC:IDC-Header_2x10_P2.54mm_Vertical, F.Cu at (141.9, 32.8)
- added L3: 3.2u, Inductor_THT:L_Toroid_Vertical_L22.4mm_W10.2mm_P7.90mm_Vishay_TJ4, F.Cu at (193.3, 63.9)
- added L4: 3.958u, Inductor_THT:L_Toroid_Vertical_L22.4mm_W10.2mm_P7.90mm_Vishay_TJ4, F.Cu at (187.8, 46.9)
- added L5: 3.2u, Inductor_THT:L_Toroid_Vertical_L22.4mm_W10.2mm_P7.90mm_Vishay_TJ4, F.Cu at (201.8, 90.2)
- added Q6: IRFZ44N, Package_TO_SOT_THT:TO-220-3_Vertical, F.Cu at (175.4, 92.2)
- added Q7: IRFP3006, Package_TO_SOT_THT:TO-247-3_Vertical, F.Cu at (203.3, 28.1)
- added Q8: MPSA42, Package_TO_SOT_THT:TO-92_Inline_Wide, F.Cu at (207.5, 37.2)
- added R1: 330k, Resistor_THT:R_Axial_DIN0207_L6.3mm_D2.5mm_P10.16mm_Horizontal, F.Cu at (22.3, 130.3)
- added R12: 910k, Resistor_THT:R_Axial_DIN0207_L6.3mm_D2.5mm_P10.16mm_Horizontal, F.Cu at (52.8, 149.8)
- added R13: 15k, Resistor_THT:R_Axial_DIN0207_L6.3mm_D2.5mm_P10.16mm_Horizontal, F.Cu at (52.8, 152.8)
- added R14: 220, Resistor_THT:R_Axial_DIN0207_L6.3mm_D2.5mm_P10.16mm_Horizontal, F.Cu at (44.9, 158.2)
- added R15: 300m, Resistor_SMD:R_2512_6332Metric_Pad1.40x3.35mm_HandSolder, F.Cu at (60.6, 145.3)
- added R16: 300m, Resistor_SMD:R_2512_6332Metric_Pad1.40x3.35mm_HandSolder, F.Cu at (60.6, 149.4)
- added R17: 300m, Resistor_SMD:R_2512_6332Metric_Pad1.40x3.35mm_HandSolder, F.Cu at (60.6, 153.4)
- added R18: 300m, Resistor_SMD:R_2512_6332Metric_Pad1.40x3.35mm_HandSolder, F.Cu at (60.6, 157.5)
- added R2: 4.7k, Resistor_THT:R_Axial_DIN0207_L6.3mm_D2.5mm_P10.16mm_Horizontal, F.Cu at (26.9, 140.5)
- added R28: 330, Resistor_THT:R_Axial_DIN0207_L6.3mm_D2.5mm_P10.16mm_Horizontal, F.Cu at (207.5, 57.5)
- added R29: 10k, Resistor_THT:R_Axial_DIN0204_L3.6mm_D1.6mm_P5.08mm_Horizontal, F.Cu at (218.6, 31.0)
- added R30: 10k, Resistor_THT:R_Axial_DIN0204_L3.6mm_D1.6mm_P5.08mm_Horizontal, F.Cu at (169.4, 92.2)
- added R31: 330, Resistor_THT:R_Axial_DIN0207_L6.3mm_D2.5mm_P10.16mm_Horizontal, F.Cu at (153.2, 90.7)
- added R32: 1/5W, Resistor_THT:R_Axial_Power_L38.0mm_W6.4mm_P40.64mm, F.Cu at (224.0, 101.6)
- added R33: 1k, Resistor_THT:R_Axial_DIN0204_L3.6mm_D1.6mm_P5.08mm_Horizontal, F.Cu at (204.3, 23.1)
- added R5: 3.3, Resistor_THT:R_Axial_DIN0207_L6.3mm_D2.5mm_P10.16mm_Horizontal, F.Cu at (42.6, 146.7)
- added REF**: MountingHole_3mm_Pad_Via, MountingHole:MountingHole_3mm_Pad_Via, F.Cu at (115.6, 23.9)
- added REF**: MountingHole_3mm_Pad_Via, MountingHole:MountingHole_3mm_Pad_Via, F.Cu at (84.7, 118.4)
- added RV1: 10k, Potentiometer_THT:Potentiometer_Bourns_3296W_Vertical, F.Cu at (23.8, 149.6)
- added U10: LM1117DT-5.0, Package_TO_SOT_SMD:TO-252-3_TabPin2, F.Cu at (134.8, 94.0)
- added U12: TLP421P, Package_DIP:DIP-4_W7.62mm, F.Cu at (210.7, 21.3)
- added U13: TLP421P, Package_DIP:DIP-4_W7.62mm, F.Cu at (154.2, 96.5)
- added U2: ICE1PCS02, Package_DIP:DIP-8_W7.62mm, F.Cu at (32.2, 145.2)
- added U7: PIC16F18455-I/SO, Package_SO:SOIC-28W_7.5x17.9mm_P1.27mm, F.Cu at (145.9, 79.1)
- C1: value 1u -> 1u/50V
- C18: renamed from C7; value 1u -> 470u/16V; footprint Capacitor_THT:CP_Radial_D4.0mm_P1.50mm -> Capacitor_THT:CP_Radial_D8.0mm_P3.50mm
- C8: renamed from C6; value 6.8u -> 6.8u/400V
- C9: renamed from C8; value 470u -> 470u/400V
- D10: renamed from D9; value S40D45C -> S60SC6MT
- D6: renamed from D5; value S30D45C -> S60SC6MT
- D7: renamed from D6; value S30D45C -> S60SC6MT
- H4: renamed from H6; value + connection to load -> +
- J5: renamed from J2; value Wire -> Wire (it's copper)
- L2: value 5u -> 3.2u; footprint Inductor_THT:L_Toroid_Vertical_L41.9mm_W19.1mm_P15.80mm_Vishay_TJ7 -> Inductor_THT:L_Toroid_Vertical_L22.4mm_W10.2mm_P7.90mm_Vishay_TJ4
- R19: renamed from R9; value 100 -> 330
- R20: renamed from R10; value 100 -> 330
- moved H4 99.7 mm to (183.1, 27.6)
- moved D6 89.2 mm to (209.3, 66.9), turned to -90 degrees
- moved C6 74.7 mm to (160.2, 140.6), turned to 45 degrees
- moved D10 68.2 mm to (209.2, 84.7), turned to -90 degrees
- moved D7 67.2 mm to (209.2, 102.5), turned to -90 degrees
- moved C5 58.0 mm to (166.6, 142.9), turned to 0 degrees
- moved C18 47.7 mm to (148.0, 112.9)
- moved U3 43.7 mm to (144.0, 66.0), turned to 180 degrees
- moved Q1 37.6 mm to (39.1, 118.6)
- moved J5 36.1 mm to (122.2, 26.9)
- moved L2 27.6 mm to (193.3, 75.9), turned to 180 degrees
- moved C8 26.5 mm to (67.8, 133.7), turned to 90 degrees
- moved REF** 17.6 mm to (161.3, 123.2)
- moved L1 16.3 mm to (37.8, 139.7), turned to 180 degrees
- moved C4 10.8 mm to (110.7, 150.0)
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- renumbered C9 to C10, C10 to C11, C11 to C12, C12 to C13, C13 to C14, C14 to C15, C15 to C16, C16 to C17, C2 to C4, C3 to C5, C4 to C6, C5 to C7, D2 to D3, D3 to D4, D4 to D5, H3 to H1, H1 to H2, H2 to H3, J3 to J4, R6 to R10, R7 to R11, R11 to R21, R12 to R22, R13 to R23, R14 to R24, R15 to R25, R16 to R26, R1 to R3, R2 to R4, R4 to R6, R5 to R7, R3 to R9, RV1 to RV2, RV2 to RV3, U2 to U4, U4 to U5, U5 to U6, U6 to U8, U7 to U9
Connections:
- net LINE renamed VAC
- net Net-(D1-+) renamed /rectified 300V
- net Net-(D1-Pad2) renamed /live filtered
- net Net-(D1-Pad4) renamed /neut filtered
- C10 pad 2: GNDD -> GND
- C11 pad 2: GNDD -> GND
- D1 pad 3: GND -> /PFC_SHUNT
- D10 pad 1: Net-(D7-A) -> /+HALF_RECT
- D10 pad 2: Net-(D9-A) -> LV_RECT
- D10 pad 3: Net-(D8-A) -> /-HALF_RECT
- D6 pad 2: Net-(D5-A) -> /+HALF_RECT
- D7 pad 2: Net-(D6-A) -> /-HALF_RECT
- H4 pad 1: VBUS -> VDC
- JP2 pad 2: Net-(JP2-B) -> 2IN+
- JP4 pad 1: VBUS -> VDC
- JP6 pad 2: Net-(JP2-B) -> 2IN+
- JP7 pad 1: VBUS -> VDC
- L2 pad 1: Net-(D9-A) -> Net-(C22-Pad1)
- L2 pad 2: VBUS -> Net-(C19-Pad1)
- R21 pad 2: GNDD -> GND
- R22 pad 2: GNDD -> GND
- RV3 pad 1: /set to 750 ohm -> unconnected-(RV3-Pad1)
- U1 pad 3: GNDD -> GND
- U3 pad 1: Net-(A1-D8) -> SPI_MOSI
- U3 pad 2: Net-(A1-D13) -> SPI_CLK
- U3 pad 3: Net-(A1-D12) -> DAC_~{CS}
- U8 pad 4: GNDD -> GND
- U9 pad 4: GNDD -> GND
Routing:
- net +12V: track 69.7 -> 274.5 mm, vias 1 -> 5
- net VDC: track 0.00 -> 166.4 mm, vias 0 -> 4
- net GND: track 82.0 -> 239.2 mm, vias 0 -> 24
- net OUTPUT_CONTROL: track 0.00 -> 152.6 mm, vias 0 -> 2
- net Net-(T1-SA): track 140.3 -> 5.08 mm
- net Net-(T1-SD): track 136.6 -> 46.3 mm
- net VBUS: track 104.8 -> 15.1 mm, vias 1 -> 0
- net +12VA: track 17.6 -> 105.9 mm, vias 0 -> 1
- net /UI_1: track 0.00 -> 84.8 mm, vias 0 -> 2
- net Net-(D5-A): track 84.4 -> 0.00 mm
- net Net-(D6-A): track 84.2 -> 0.00 mm
- net /UI_0: track 0.00 -> 79.9 mm, vias 0 -> 2
- net GND1: track 341.7 -> 265.2 mm, vias 5 -> 11
- net /7SEG_A: track 0.00 -> 75.6 mm, vias 0 -> 2
- net /7SEG_D: track 0.00 -> 73.5 mm, vias 0 -> 2
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- added copper zone on B.Cu, net +5V
- added copper zone on B.Cu, net /+HALF_RECT
- added copper zone on F.Cu, net /+HALF_RECT
- added copper zone on B.Cu, net /-HALF_RECT
- added copper zone on F.Cu, net /-HALF_RECT
- added copper zone on B.Cu, net /PFC_SHUNT
- added copper zone on F.Cu, net GND1
- added copper zone on B.Cu, net LV_RECT
- added copper zone on F.Cu, net LV_RECT
- added copper zone on F.Cu, net NEUT
- added copper zone on F.Cu, net Net-(C19-Pad1)
- added copper zone on F.Cu, net Net-(C20-Pad1)
- added copper zone on B.Cu, net Net-(C22-Pad1)
- added copper zone on F.Cu, net Net-(C22-Pad1)
- added copper zone on F.Cu, net Net-(D3-A)
- added copper zone on B.Cu, net Net-(Q4-S)
- added copper zone on B.Cu, net VDC
- added copper zone on F.Cu, net VDC
- removed copper zone on B.Cu, net GNDD
- removed copper zone on B.Cu, net Net-(C17-Pad2)
- removed copper zone on B.Cu, net Net-(D5-A)
- removed copper zone on F.Cu, net Net-(D5-A)
- removed copper zone on B.Cu, net Net-(D6-A)
- removed copper zone on F.Cu, net Net-(D6-A)
- removed copper zone on B.Cu, net Net-(D7-A)
- removed copper zone on F.Cu, net Net-(D7-A)
- removed copper zone on B.Cu, net Net-(D8-A)
- removed copper zone on F.Cu, net Net-(D8-A)
- removed copper zone on B.Cu, net Net-(D9-A)
- removed copper zone on F.Cu, net Net-(D9-A)
Other:
- outline, holes or cut-outs redrawn
- board text added: "12V EXT INPUT"
- board text removed: "12V PSU INPUT"
- board text removed: "AC INPUT FILTER"
- board text removed: "HV BUFFER CAP"
- board text removed: "LV BUFFER CAP"
- board text removed: "PFC SECTION"
- board text removed: "RESONANCE CAPACITORS"

Commit message: Add files via upload
Close to finish
Parts:
- R32: footprint Resistor_THT:R_Axial_Power_L38.0mm_W6.4mm_P40.64mm -> Resistor_THT:R_Axial_Power_L20.0mm_W6.4mm_P25.40mm
- moved R32 45.7 mm to (179.2, 93.0), turned to -90 degrees
- moved R12 3.11 mm to (52.7, 152.9)
- moved R13 2.98 mm to (52.8, 149.9)
- moved R29 0.90 mm to (217.7, 31.1)
- moved R33 0.25 mm to (204.3, 23.4)
Routing:
- net Net-(Q6-D): track 0.00 -> 5.72 mm
- net 300V clean: track 185.1 -> 183.8 mm
- net Net-(Q6-G): track 35.9 -> 35.0 mm
- net BUZZER: track 60.6 -> 61.5 mm
- net GND1: track 265.2 -> 265.9 mm
- net VBUS: vias 0 -> 6
- added copper zone on B.Cu, net +12V
- added copper zone on B.Cu, net Net-(D11-K)
- added copper zone on B.Cu, net Net-(D12-K)
- added copper zone on F.Cu, net Net-(D12-K)
- added copper zone on F.Cu, net Net-(Q8-B)

Commit message: Add files via upload
Parts:
- added C31: 1u/50V, Capacitor_THT:CP_Radial_D4.0mm_P1.50mm, F.Cu at (153.6, 87.4)
- added C32: 1u, Capacitor_THT:CP_Radial_D4.0mm_P1.50mm, F.Cu at (119.1, 118.6)
- added C33: 1u, Capacitor_THT:CP_Radial_D4.0mm_P1.50mm, F.Cu at (129.2, 71.2)
- moved C29 8.54 mm to (203.7, 51.4), turned to 90 degrees
- moved R31 3.56 mm to (156.7, 90.6)
- moved R28 2.47 mm to (209.9, 57.0)
- moved D12 2.16 mm to (209.7, 43.9), turned to 0 degrees
- moved REF** 0.87 mm to (160.4, 123.3)
- moved Q8 0.51 mm to (207.5, 36.7)
- moved C24 0.17 mm to (202.1, 44.3)
Connections:
- U3 pad 6: Net-(U3-REF) -> REF
- U4 pad 13: Net-(U4-OUTCTRL) -> REF
- U4 pad 14: Net-(U4-OUTCTRL) -> REF
Routing:
- net REF: track 0.00 -> 69.4 mm, vias 0 -> 3
- net GND1: track 265.9 -> 286.9 mm, vias 11 -> 15
- net +12V: track 274.5 -> 289.4 mm, vias 5 -> 3
- net VDC: track 166.8 -> 178.0 mm
- net Net-(D11-K): track 31.8 -> 41.5 mm, vias 0 -> 3
- net Net-(C19-Pad1): track 27.3 -> 31.5 mm
- net VPP: track 37.6 -> 40.6 mm
- net SPI_CLK: track 59.5 -> 56.8 mm, vias 2 -> 0
- net Net-(U4-OUTCTRL): track 2.54 -> 0.00 mm
- net Net-(D12-K): track 30.9 -> 29.0 mm
- net OUT_A: track 52.8 -> 54.2 mm
- net SPI_MOSI: track 55.4 -> 56.7 mm
- net Net-(U4-C2): track 14.7 -> 15.8 mm
- net Net-(Q8-B): track 16.9 -> 15.9 mm
- net 2IN+: track 53.3 -> 52.5 mm
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- added copper zone on F.Cu, net Net-(D11-K)
- added copper zone on B.Cu, net Net-(R28-Pad1)
- removed copper zone on F.Cu, net Net-(D12-K)
Other:
- outline, holes or cut-outs redrawn

Commit message: Add files via upload
Parts:
- removed C33: 1u, Capacitor_THT:CP_Radial_D4.0mm_P1.50mm
- removed D10, D6, D7: S60SC6MT, Package_TO_SOT_THT:TO-247-3_Vertical
- removed H1: EARTH, MountingHole:MountingHole_6mm_Pad
- removed H2: LIVE, MountingHole:MountingHole_6mm_Pad
- removed H3: NEUTRAL, MountingHole:MountingHole_6mm_Pad
- removed JP3, JP4, JP5, JP6: A, Jumper:SolderJumper-2_P1.3mm_Open_RoundedPad1.0x1.5mm
- removed JP7, JP8: B, Jumper:SolderJumper-2_P1.3mm_Open_RoundedPad1.0x1.5mm
- added ?: , , F.Cu at (179.8, 120.1)
- added D13: IN4002, Diode_THT:D_A-405_P7.62mm_Horizontal, F.Cu at (70.6, 79.5)
- added D14: IN4002, Diode_THT:D_A-405_P7.62mm_Horizontal, F.Cu at (66.0, 98.6)
- added D15: IN4002, Diode_THT:D_A-405_P7.62mm_Horizontal, F.Cu at (70.1, 116.3)
- added D8: RUN, LED_THT:LED_D3.0mm, F.Cu at (153.0, 98.4)
- added D9: IN4002, Diode_THT:D_A-405_P7.62mm_Horizontal, F.Cu at (55.6, 55.4)
- added J1: C14 socket, Calibration_Scale:C14 AC socket, F.Cu at (159.3, 147.3)
- added Q10: IRFP4321, Package_TO_SOT_THT:TO-247-3_Vertical, F.Cu at (174.0, 50.0)
- added Q9: IRFP4321, Package_TO_SOT_THT:TO-247-3_Vertical, F.Cu at (174.0, 94.0)
- added R34: 330, Resistor_THT:R_Axial_DIN0207_L6.3mm_D2.5mm_P7.62mm_Horizontal, F.Cu at (138.3, 77.1)
- added R35: 1k, Resistor_THT:R_Axial_DIN0204_L3.6mm_D1.6mm_P5.08mm_Horizontal, F.Cu at (141.7, 99.6)
- added R36: 10k, Resistor_THT:R_Axial_DIN0204_L3.6mm_D1.6mm_P5.08mm_Horizontal, F.Cu at (123.7, 91.9)
- added R37: 1k, Resistor_THT:R_Axial_DIN0204_L3.6mm_D1.6mm_P5.08mm_Horizontal, F.Cu at (181.1, 54.4)
- added R38: 22, Resistor_THT:R_Axial_DIN0207_L6.3mm_D2.5mm_P7.62mm_Horizontal, F.Cu at (129.5, 88.4)
- added R39: 1k, Resistor_THT:R_Axial_DIN0204_L3.6mm_D1.6mm_P5.08mm_Horizontal, F.Cu at (173.7, 89.2)
- added R40: 470, Resistor_THT:R_Axial_DIN0204_L3.6mm_D1.6mm_P5.08mm_Horizontal, F.Cu at (166.4, 44.2)
- added R41: 470, Resistor_THT:R_Axial_DIN0204_L3.6mm_D1.6mm_P5.08mm_Horizontal, F.Cu at (158.5, 88.6)
- added REF**: OSHW-Logo2_7.3x6mm_SilkScreen, Symbol:OSHW-Logo2_7.3x6mm_SilkScreen, F.Cu at (194.6, 125.5)
- added REF**: MountingHole_2.2mm_M2_DIN965_Pad, MountingHole:MountingHole_2.2mm_M2_DIN965_Pad, F.Cu at (179.8, 66.3)
- added RV4: 10k, Potentiometer_THT:Potentiometer_Bourns_3296W_Vertical, F.Cu at (118.6, 118.4)
- added SW1: SW_Push, Button_Switch_SMD:SW_Push_1P1T_NO_CK_KSC6xxJ, F.Cu at (130.6, 75.2)
- added U14: NE5532, Package_DIP:DIP-8_W7.62mm, F.Cu at (118.4, 114.0)
- added U15: TLP421P, Package_DIP:DIP-4_W7.62mm, F.Cu at (161.9, 47.6)
- added U16: TLP421P, Package_DIP:DIP-4_W7.62mm, F.Cu at (150.5, 92.1)
- C32: value 1u -> 1u/50V
- C7: value 10n -> 1n
- J2: footprint Connector_PinHeader_2.54mm:PinHeader_1x06_P2.54mm_Vertical -> Connector_PinHeader_2.54mm:PinHeader_2x04_P2.54mm_Vertical
- JP1, JP2: value B -> SolderJumper_2_Open; footprint Jumper:SolderJumper-2_P1.3mm_Open_RoundedPad1.0x1.5mm -> Jumper:SolderJumper-2_P1.3mm_Open_TrianglePad1.0x1.5mm
- R10, RV3: value 1k -> 10k
- R11: value 100k -> 22; footprint Resistor_THT:R_Axial_DIN0207_L6.3mm_D2.5mm_P10.16mm_Horizontal -> Resistor_THT:R_Axial_DIN0207_L6.3mm_D2.5mm_P7.62mm_Horizontal
- R19, R20: value 330 -> 470; footprint Resistor_THT:R_Axial_DIN0207_L6.3mm_D2.5mm_P10.16mm_Horizontal -> Resistor_THT:R_Axial_DIN0204_L3.6mm_D1.6mm_P5.08mm_Horizontal
- R25: footprint Resistor_THT:R_Axial_DIN0207_L6.3mm_D2.5mm_P10.16mm_Horizontal -> Resistor_THT:R_Axial_DIN0207_L6.3mm_D2.5mm_P15.24mm_Horizontal
- R3: value 100k -> 330k; footprint Resistor_THT:R_Axial_DIN0207_L6.3mm_D2.5mm_P10.16mm_Horizontal -> Resistor_THT:R_Axial_DIN0207_L6.3mm_D2.5mm_P7.62mm_Horizontal
- R4: value 500 -> 560k; footprint Resistor_THT:R_Axial_DIN0207_L6.3mm_D2.5mm_P10.16mm_Horizontal -> Resistor_THT:R_Axial_DIN0207_L6.3mm_D2.5mm_P7.62mm_Horizontal
- R6: value 1k -> 36k; footprint Resistor_THT:R_Axial_DIN0204_L3.6mm_D1.6mm_P5.08mm_Horizontal -> Resistor_THT:R_Axial_DIN0207_L6.3mm_D2.5mm_P7.62mm_Horizontal
- R7: value 100k -> 6.8k; footprint Resistor_THT:R_Axial_DIN0207_L6.3mm_D2.5mm_P10.16mm_Horizontal -> Resistor_THT:R_Axial_DIN0207_L6.3mm_D2.5mm_P7.62mm_Horizontal
- R9: value 500 -> 5.1k; footprint Resistor_THT:R_Axial_DIN0207_L6.3mm_D2.5mm_P10.16mm_Horizontal -> Resistor_THT:R_Axial_DIN0207_L6.3mm_D2.5mm_P7.62mm_Horizontal
- U7: value PIC16F18455-I/SO -> AVR64DA32x-xPT; footprint Package_SO:SOIC-28W_7.5x17.9mm_P1.27mm -> Package_QFP:TQFP-32_7x7mm_P0.8mm
- moved BZ1 84.7 mm to (153.7, 45.1), turned to 90 degrees
- moved JP2 64.9 mm to (178.1, 40.6), turned to 180 degrees
- moved C32 53.0 mm to (141.7, 70.6), turned to -90 degrees
- moved R4 50.7 mm to (128.3, 114.0), turned to 180 degrees
- moved JP1 41.8 mm to (165.9, 91.9), turned to 180 degrees
- moved R11 41.1 mm to (136.5, 67.1), turned to 180 degrees
- moved R31 35.8 mm to (181.6, 116.3)
- moved C26 35.0 mm to (212.4, 58.9), turned to 0 degrees
- moved C20 34.9 mm to (212.4, 68.1), turned to 0 degrees
- moved C19 34.9 mm to (212.4, 77.2), turned to 0 degrees
- moved C27 34.8 mm to (212.4, 86.4), turned to 0 degrees
- moved R20 28.0 mm to (115.8, 103.4), turned to 180 degrees
- moved R6 27.1 mm to (110.2, 67.2), turned to 0 degrees
- moved C18 25.4 mm to (169.9, 125.8), turned to -135 degrees
- moved C6 23.5 mm to (183.4, 136.6), turned to -90 degrees
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Connections:
- net Net-(C19-Pad1) renamed /FILTER2
- net Net-(C20-Pad1) renamed /FILTER3
- net Net-(C4-Pad1) renamed /LIVE_FUSED
- net Net-(U4-C1) renamed /S-
- net Net-(U4-C2) renamed /S+
- net Net-(U8-HIN) renamed /DRIVE_1
- net Net-(U8-LIN) renamed /DRIVE_2
- net REF renamed DAC_REF
- C22 pad 1: Net-(C22-Pad1) -> /FILTER1
- C28 pad 1: Net-(C22-Pad1) -> /FILTER1
- C31 pad 1: VPP -> +5V
- C32 pad 1: +12V -> +5V
- J2 pad 1: VPP -> SPI_MISO
- J2 pad 3: GND1 -> SPI_CLK
- J2 pad 4: ICSPDAT -> SPI_MOSI
- J2 pad 5: ICSPCLK -> ~{RESET}
- J2 pad 6: unconnected-(J2-Pin_6-Pad6) -> GND1
- J3 pad 11: /UI_1 -> UI_1
- J3 pad 9: /UI_0 -> UI_0
- JP1 pad 1: OUT_A -> Net-(JP1-A)
- JP2 pad 2: 2IN+ -> Net-(JP2-B)
- L2 pad 1: Net-(C22-Pad1) -> /FILTER1
- L5 pad 2: Net-(C22-Pad1) -> /FILTER1
- R1 pad 1: 300V clean -> /rectified 300V
- R10 pad 1: Net-(JP3-B) -> Net-(U4-2IN-)
- R10 pad 2: Net-(U4-1IN-) -> Net-(U4-FB)
- R11 pad 1: Net-(U4-1IN-) -> DAC_CUR
- R11 pad 2: Net-(U4-FB) -> Net-(U4-2IN-)
- R19 pad 1: Net-(U4-E2) -> +12V
- R19 pad 2: GND1 -> Net-(R19-Pad2)
- R20 pad 1: Net-(U4-E1) -> +12V
- R20 pad 2: GND1 -> Net-(R20-Pad2)
- R3 pad 2: OUT_B -> VBUS
- R32 pad 2: VBUS -> /FILTER1
- R4 pad 2: GND1 -> ADC_CUR
- R6 pad 1: Net-(JP5-B) -> GND1
- R6 pad 2: Net-(U4-2IN-) -> Net-(R6-Pad2)
- R7 pad 1: Net-(U4-FB) -> GND1
- R7 pad 2: Net-(U4-2IN-) -> Net-(R7-Pad2)
- RV2 pad 2: Net-(JP2-A) -> ADC_VOL
- RV2 pad 3: Net-(R4-Pad1) -> Net-(R6-Pad2)
- T1 pad 3: Net-(T1-SA) -> /+HALF_RECT
- T1 pad 4: GND1 -> LV_RECT
- T1 pad 5: GND1 -> LV_RECT
- T1 pad 6: Net-(T1-SD) -> /-HALF_RECT
- U3 pad 4: OUT_A -> DAC_VOL
- U3 pad 7: OUT_B -> DAC_CUR
- U4 pad 1: Net-(JP1-B) -> ADC_VOL
- U4 pad 10: Net-(U4-E2) -> GND1
- U4 pad 16: 2IN+ -> ADC_CUR
- U4 pad 9: Net-(U4-E1) -> GND1
- U5 pad 1: +5V -> Net-(R19-Pad2)
- U6 pad 1: +5V -> Net-(R20-Pad2)
- U7 pad 1: VPP -> ADC_CUR
- U7 pad 10: /7SEG_DEMUX_C -> /7SEG_DEMUX_A
- U7 pad 11: OUTPUT_CONTROL -> /7SEG_DEMUX_B
- U7 pad 12: FAN_PWM -> /7SEG_DEMUX_C
- U7 pad 13: UI_3 -> /7SEG_DEMUX_D
- U7 pad 14: SPI_CLK -> /7SEG_A
- U7 pad 15: DAC_~{CS} -> /7SEG_B
- U7 pad 16: SPI_MOSI -> /7SEG_C
- U7 pad 17: DISPLAY_~{CS} -> /7SEG_D
- U7 pad 18: UI_2 -> +5V
- U7 pad 2: ADC0 -> SPI_MOSI
- U7 pad 20: +5V -> unconnected-(U7-XTAL32K1/PF0-Pad20)
- U7 pad 21: /7SEG_A -> unconnected-(U7-XTAL32K2/PF1-Pad21)
- U7 pad 22: /7SEG_B -> OUTPUT_CONTROL
- U7 pad 23: /7SEG_C -> FAN_PWM
- U7 pad 24: /7SEG_D -> Net-(U7-PF4)
- U7 pad 25: /UI_0 -> DISPLAY_~{CS}
- U7 pad 26: /UI_1 -> ~{RESET}
- U7 pad 27: ICSPCLK -> UPDI
- U7 pad 28: ICSPDAT -> +5V
- U7 pad 3: ADC1 -> SPI_MISO
- U7 pad 4: CROWBAR -> SPI_CLK
- U7 pad 5: BUZZER -> DAC_~{CS}
- U7 pad 6: /7SEG_DEMUX_A -> UI_0
- U7 pad 7: /7SEG_DEMUX_B -> UI_1
- U7 pad 8: GND1 -> UI_2
- U7 pad 9: /7SEG_DEMUX_D -> UI_3
Routing:
- net VDC: track 178.0 -> 65.3 mm, vias 4 -> 1
- net /S-: track 29.0 -> 136.7 mm, vias 0 -> 5
- net VBUS: track 15.2 -> 113.6 mm, vias 5 -> 1
- net /UI_1: track 84.8 -> 0.00 mm, vias 2 -> 0
- net +12V: track 289.4 -> 372.6 mm, vias 3 -> 7
- net /UI_0: track 79.9 -> 0.00 mm, vias 2 -> 0
- net ADC_CUR: track 0.00 -> 72.5 mm, vias 0 -> 3
- net UI_1: track 0.00 -> 65.6 mm, vias 0 -> 2
- net UI_0: track 0.00 -> 65.6 mm, vias 0 -> 2
- net ADC_VOL: track 0.00 -> 57.5 mm, vias 0 -> 2
- net OUT_A: track 54.2 -> 0.00 mm, vias 4 -> 0
- net GND1: track 286.9 -> 234.0 mm, vias 15 -> 11
- net 2IN+: track 52.5 -> 0.00 mm, vias 1 -> 0
- net SPI_CLK: track 56.8 -> 107.5 mm, vias 0 -> 5
- net ~{RESET}: track 0.00 -> 47.1 mm, vias 0 -> 3
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- added copper zone on F.Cu, net /FILTER1
- added copper zone on F.Cu, net VAC
- removed copper zone on B.Cu, net +12V
- removed copper zone on B.Cu, net +5V
- removed copper zone on B.Cu, net /+HALF_RECT
- removed copper zone on B.Cu, net /-HALF_RECT
- removed copper zone on F.Cu, net GND1
- removed copper zone on B.Cu, net LV_RECT
- removed copper zone on B.Cu, net Net-(C22-Pad1)
- removed copper zone on F.Cu, net Net-(C22-Pad1)
- removed copper zone on B.Cu, net Net-(D11-K)
- removed copper zone on F.Cu, net Net-(D11-K)
- removed copper zone on B.Cu, net Net-(D12-K)
- removed copper zone on F.Cu, net Net-(Q8-B)
- removed copper zone on B.Cu, net Net-(R28-Pad1)
- removed copper zone on B.Cu, net Net-(T1-SA)
- removed copper zone on F.Cu, net Net-(T1-SA)
- removed copper zone on B.Cu, net Net-(T1-SD)
- removed copper zone on F.Cu, net Net-(T1-SD)
Other:
- outline, holes or cut-outs redrawn
- board text added: "+5V"
- board text added: "19.09.2023 SuperSMPS v2.1 M. Czarnecki Prototype JLCJLCJLCJLC"
- board text added: "GND"
- board text added: "MISO"
- board text added: "MOSI"
- board text added: "RST"
- board text added: "SCK"
- board text added: "UPDI"
